Commit message: 자율주행에 맞는 카메라 setting

File: zed_wrapper/urdf/zed_macro.urdf.xacro (robot description, xacro)
@@ -83,4 +83,10 @@
     <!-- Camera mounting point (the threaded screw hole in the bottom) -->
     <link name="${name}_camera_link" />
+    <!-- <link name="${name}_robot_base" />
+    <joint name="${name}_robot_base_joint" type="fixed">
+      <parent link="${name}_camera_link"/>
+      <child link="${name}_robot_base"/>
+      <origin xyz="0 0 0" rpy="0 0 0"/>
+    </joint> -->
     <!-- Camera Center -->
     <link name="${name}_camera_center">
